Commit message: add realsense pkg and update sensor record part

File: cartographer_detailed_comments_ws/src/cartographer_ros/cartographer_ros/urdf/online_2d.urdf (robot description, URDF)
Before this commit: robot online_slam_3d, 3 links, 1 joints
Joints:
- removed joint LiDAR_to_imu
- added joint LiDAR_to_pixhawk: type fixed, parent base_link, child velodyne, origin xyz=0.0 0.0 0.17 rpy=0. 0. 0.
- added joint imu_to_pixhawk: type fixed, parent base_link, child imu_link, origin xyz=0.0 0.0 0.06 rpy=0. 0. 0
