Commit message: on/off record data

File: cartographer_detailed_comments_ws/src/cartographer_ros/cartographer_ros/urdf/online_3d.urdf (robot description, URDF)
Before this commit: robot online_slam_3d, 3 links, 2 joints
Links:
- added link camera_link; visual box size=0.090 0.025 0.025
Joints:
- added joint camera_to_pixhawk: type fixed, parent base_link, child camera_link, origin xyz=0.0 0.0 0.06 rpy=0. 0. 0
