Commit message: update offline 3d(real-time), fix 'z drift'

File: cartographer_detailed_comments_ws/src/cartographer_ros/cartographer_ros/urdf/offline_2d.urdf (robot description, URDF)
Before this commit: robot online_slam_3d, 3 links, 2 joints
Links:
- added link camera_link; visual box size=0.090 0.025 0.025
- link base_link: geometry 
Joints:
- removed joint LiDAR_to_pixhawk
- removed joint imu_to_pixhawk
- added joint LiDAR_to_base: type fixed, parent base_link, child velodyne, origin xyz=0.0 0.0 0.13104 rpy=0. 0. 0.
- added joint camera_to_base: type fixed, parent base_link, child camera_link, origin xyz=-0.0175 0.0765 0.0125 rpy=0. 0. 0.
- added joint imu_to_base: type fixed, parent base_link, child imu_link, origin xyz=0.0 0.0 0.0 rpy=0. 0. 0.

File: cartographer_detailed_comments_ws/src/cartographer_ros/cartographer_ros/urdf/online_3d.urdf (robot description, URDF)
Before this commit: robot online_slam_3d, 4 links, 3 joints
Links:
- link base_link: geometry 
Joints:
- removed joint LiDAR_to_pixhawk
- removed joint camera_to_pixhawk
- removed joint imu_to_pixhawk
- added joint LiDAR_to_base: type fixed, parent base_link, child velodyne, origin xyz=0.0 0.0 0.13104 rpy=0. 0. 0.
- added joint camera_to_base: type fixed, parent base_link, child camera_link, origin xyz=-0.0175 0.0765 0.0125 rpy=0. 0. 0.
- added joint imu_to_base: type fixed, parent base_link, child imu_link, origin xyz=0.0 0.0 0.0 rpy=0. 0. 0.

Commit message: 240130

File: cartographer_detailed_comments_ws/src/cartographer_ros/cartographer_ros/urdf/offline_2d.urdf (robot description, URDF)
Before this commit: robot online_slam_3d, 4 links, 3 joints
Joints:
- joint LiDAR_to_base: origin xyz=0.0 0.0 0.13104 rpy=0. 0. 0. -> xyz=0.0 0.0 0.13304 rpy=0. 0. 0.
- joint camera_to_base: origin xyz=-0.0175 0.0765 0.0125 rpy=0. 0. 0. -> xyz=0.0325 -0.092 0.02274 rpy=-1.5707963 0. 3.1415926
